File: CESE-7Co2018_DCI.kicad_pcb (KiCad board)
At the start: 2 copper layers, 138 x 87 mm, 78 parts, among them J1 Electrodes, J2 Power, J3 PreOUT1, J4 PreOUT2, J5 OUT, SW1 Differential_Gain, SW2 LowCuteoff_C, SW3 LowCuteoff_R, SW4 HighCuteoff_C, SW5 HighCuteoff_R, SW6 Filter_Gain, SW7 DRL_EN, SW8 Offset_EN, U1 AD620, U2 LM741, U3 LM741, U4 LM741, U5 LM741

Commit message: Con todas las correcciones recomendadas
Parts:
- added D1: Green Led, LED_THT:LED_D5.0mm, F.Cu at (49.0, 69.0)
- added D2: Blue Led, LED_THT:LED_D5.0mm, F.Cu at (49.0, 76.5)
- JP1, JP10, JP2, JP3, JP4, JP5, JP6, JP7, JP8, JP9: footprint Connector_PinHeader_1.00mm:PinHeader_1x02_P1.00mm_Vertical -> Connector_PinHeader_2.54mm:PinHeader_1x02_P2.54mm_Vertical
- moved JP5 2.57 mm to (107.8, 88.8)
- moved JP6 2.25 mm to (107.8, 92.5)
- moved JP9 1.60 mm to (138.0, 99.8)
- moved JP3 1.46 mm to (45.8, 106.8)
- moved JP7 1.27 mm to (118.3, 99.8)
- moved JP1 1.25 mm to (85.6, 88.8)
- moved JP10 1.00 mm to (138.0, 103.5)
- moved JP4 0.75 mm to (45.8, 103.0)
- moved JP8 0.25 mm to (118.3, 103.5)
Connections:
- J1 pad R: IN- -> IN+
- J1 pad S: IN+ -> IN-
- U1 pad 2: IN+ -> IN-
- U1 pad 3: IN- -> IN+
Routing:
- net +12V: track 240.3 -> 253.0 mm
- net IN-: track 24.5 -> 36.7 mm
- net IN+: track 36.2 -> 24.7 mm
- net Net-(C5-Pad1): track 59.0 -> 64.2 mm
- net S1: track 97.7 -> 101.0 mm
- net Net-(JP1-Pad2): track 23.4 -> 20.7 mm
- net Net-(C10-Pad1): track 61.5 -> 59.2 mm
- net A1: track 67.0 -> 69.2 mm, vias 2 -> 1
- net A3: track 76.7 -> 78.7 mm
- net Net-(JP7-Pad2): track 20.0 -> 18.0 mm
- net DRL: track 33.4 -> 31.5 mm
- net A2: track 53.7 -> 55.5 mm
- net Net-(C2-Pad2): track 19.1 -> 20.7 mm
- net Net-(C2-Pad1): track 49.0 -> 50.2 mm
- net -12V: track 207.7 -> 208.8 mm
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Other:
- net class Default: clearance 0.2 -> 0.6
- rule trace_clearance: 0.2 -> 0.6
- board text added: "+12 V"
- board text added: "-12 V"
- board text added: "GND"
- board text added: "Power"
