File: CESE-7Co2018_DCI.sch (KiCad schematic (older format))
At the start: 78 parts, among them J1 OUT, J2 Power, J3 PreOUT1, J4 Electrodes, J5 PreOUT2, SW1 Differential_Gain, SW2 LowCuteoff_C, SW3 LowCuteoff_R, SW4 HighCuteoff_C, SW5 HighCuteoff_R, SW6 Filter_Gain, SW7 DRL_EN, SW8 Offset_EN, U1 AD620, U2 LM741, U3 LM741, U4 LM741, U5 LM741

Commit message: Correcciones de la primera revision de Lucianna FA
Parts:
- U1, U2, U3, U4, U5: footprint Package_DIP:DIP-8_W7.62mm -> Package_DIP:DIP-8_W7.62mm_Socket
Other:
- note added: "Los valores correspondientes a las resistencias y \ncapacitores ubicados en los selectores SW1 a SW6\nno están definidas. El docente o profesor a cargo \nde la clase será quien determine el valor de las \nmismas según sus necesidades."

Commit message: PCB Completo
Parts:
- renumbered J4 to J1, J5 to J4, J1 to J5, R14 to R10, R17 to R11, R19 to R12, R20 to R13, R21 to R14, R27 to R15, R22 to R16, R23 to R17, R24 to R18, R25 to R19, R26 to R20, R28 to R21, R29 to R22, R16 to R23, R30 to R24, R31 to R25, R18 to R26, R3 to R27, R4 to R28, R11 to R29, R5 to R3, R6 to R30, R7 to R31, R8 to R4, R9 to R5, R10 to R6, R13 to R7, R12 to R8, R15 to R9

Commit message: Con todas las correcciones recomendadas
Parts:
- added D1: Green Led, LED_THT:LED_D5.0mm, symbol Device:LED
- added D2: Blue Led, LED_THT:LED_D5.0mm, symbol Device:LED
- JP1, JP10, JP2, JP3, JP4, JP5, JP6, JP7, JP8, JP9: footprint Connector_PinHeader_1.00mm:PinHeader_1x02_P1.00mm_Vertical -> Connector_PinHeader_2.54mm:PinHeader_1x02_P2.54mm_Vertical
Connections:
- net +12V: now also D1.2 (A)
- net -12V: now also D2.1 (K)
- net GND: now also D1.1 (K), D2.2 (A)
- net IN+: now also J1.R, U1.3 (+); no longer J1.S, U1.2 (-)
- net IN-: now also J1.S, U1.2 (-); no longer J1.R, U1.3 (+)
Other:
- note added: "AD620\nManufacturer: Analogic Devices\nPackage: Lead Plastic Dual In-Line"
- note added: "Indicator Leds"
- note added: "LM741\nManufacturer: Fairchild Semiconductor\nPackage: Lead Plastic Dual In-Line"
Changed lines of the file:
@@
 encoding utf-8
 Sheet 1 1
-Title "Trabajo Final de Diseño de Circuitos Impresos"
+Title "Amplificador Biológico Educativo"
 Date "2019-05-27"
-Rev "Lucianna FA"
+Rev "1.1"
 Comp "Pizá, Alvaro Gabriel"
 Comment1 "CESE - UBA"
 Comment2 "7maCo2018"
-Comment3 ""
-Comment4 ""
+Comment3 "Revisores: Lucianna FA, Brengi D"
+Comment4 "Licencia Creative Commons Attributions Share-Alike 4.0"
 $EndDescr
 Text GLabel 5100 3175 2    50   Input ~ 0
@@
 $EndComp
 Text GLabel 5875 7100 2    50   Input ~ 0
+IN-
+Text GLabel 5875 7275 2    50   Input ~ 0
 IN+
-Text GLabel 5875 7275 2    50   Input ~ 0
-IN-
 Text GLabel 5875 7450 2    50   Input ~ 0
 DRL
@@
 F 0 "JP9" H 10375 3864 50  0000 C CNN
 F 1 "Bandpass_Bridge" H 10375 3773 50  0000 C CNN
-F 2 "Connector_PinHeader_1.00mm:PinHeader_1x02_P1.00mm_Vertical" H 10375 3600 50  0001 C CNN
+F 2 "Connector_PinHeader_2.54mm:PinHeader_1x02_P2.54mm_Vertical" H 10375 3600 50  0001 C CNN
 F 3 "~" H 10375 3600 50  0001 C CNN
 	1    10375 3600
@@
 F 0 "JP10" H 10375 3718 50  0000 C CNN
 F 1 "Bandpass_Filter" H 10375 3627 50  0000 C CNN
-F 2 "Connector_PinHeader_1.00mm:PinHeader_1x02_P1.00mm_Vertical" H 10375 3850 50  0001 C CNN
+F 2 "Connector_PinHeader_2.54mm:PinHeader_1x02_P2.54mm_Vertical" H 10375 3850 50  0001 C CNN
 F 3 "~" H 10375 3850 50  0001 C CNN
 	1    10375 3850
@@
 F 0 "JP8" H 6400 3393 50  0000 C CNN
 F 1 "Bandpass_Filter" H 6400 3302 50  0000 C CNN
-F 2 "Connector_PinHeader_1.00mm:PinHeader_1x02_P1.00mm_Vertical" H 6400 3525 50  0001 C CNN
+F 2 "Connector_PinHeader_2.54mm:PinHeader_1x02_P2.54mm_Vertical" H 6400 3525 50  0001 C CNN
 F 3 "~" H 6400 3525 50  0001 C CNN
 	1    6400 3525
@@
 F 0 "JP7" H 6400 3589 50  0000 C CNN
 F 1 "Bandpass_Bridge" H 6400 3498 50  0000 C CNN
-F 2 "Connector_PinHeader_1.00mm:PinHeader_1x02_P1.00mm_Vertical" H 6400 3325 50  0001 C CNN
+F 2 "Connector_PinHeader_2.54mm:PinHeader_1x02_P2.54mm_Vertical" H 6400 3325 50  0001 C CNN
 F 3 "~" H 6400 3325 50  0001 C CNN
 	1    6400 3325
@@
 S1
 Text GLabel 900  1650 0    50   Input ~ 0
+IN+
+Text GLabel 900  1425 0    50   Input ~ 0
 IN-
-Text GLabel 900  1425 0    50   Input ~ 0
-IN+
 $Comp
 L power:-12V #PWR0108
@@
 F 0 "JP2" H 1400 3143 50  0000 C CNN
 F 1 "Notch_Filter" H 1400 3052 50  0000 C CNN
-F 2 "Connector_PinHeader_1.00mm:PinHeader_1x02_P1.00mm_Vertical" H 1400 3275 50  0001 C CNN
+F 2 "Connector_PinHeader_2.54mm:PinHeader_1x02_P2.54mm_Vertical" H 1400 3275 50  0001 C CNN
 F 3 "~" H 1400 3275 50  0001 C CNN
 	1    1400 3275
@@
 F 0 "JP1" H 1400 3339 50  0000 C CNN
 F 1 "Notch_Bridge" H 1400 3248 50  0000 C CNN
-F 2 "Connector_PinHeader_1.00mm:PinHeader_1x02_P1.00mm_Vertical" H 1400 3075 50  0001 C CNN
+F 2 "Connector_PinHeader_2.54mm:PinHeader_1x02_P2.54mm_Vertical" H 1400 3075 50  0001 C CNN
 F 3 "~" H 1400 3075 50  0001 C CNN
 	1    1400 3075
@@
 F 0 "JP6" H 4600 3143 50  0000 C CNN
 F 1 "Notch_Filter" H 4600 3052 50  0000 C CNN
-F 2 "Connector_PinHeader_1.00mm:PinHeader_1x02_P1.00mm_Vertical" H 4600 3275 50  0001 C CNN
+F 2 "Connector_PinHeader_2.54mm:PinHeader_1x02_P2.54mm_Vertical" H 4600 3275 50  0001 C CNN
 F 3 "~" H 4600 3275 50  0001 C CNN
 	1    4600 3275
@@
 F 0 "JP4" H 3675 5575 50  0000 C CNN
 F 1 "RefToGND" H 3675 5500 50  0000 C CNN
-F 2 "Connector_PinHeader_1.00mm:PinHeader_1x02_P1.00mm_Vertical" H 3675 5650 50  0001 C CNN
+F 2 "Connector_PinHeader_2.54mm:PinHeader_1x02_P2.54mm_Vertical" H 3675 5650 50  0001 C CNN
 F 3 "~" H 3675 5650 50  0001 C CNN
 	1    3675 5650
@@
 F 0 "JP5" H 4600 3339 50  0000 C CNN
 F 1 "Notch_Bridge" H 4600 3248 50  0000 C CNN
-F 2 "Connector_PinHeader_1.00mm:PinHeader_1x02_P1.00mm_Vertical" H 4600 3075 50  0001 C CNN
+F 2 "Connector_PinHeader_2.54mm:PinHeader_1x02_P2.54mm_Vertical" H 4600 3075 50  0001 C CNN
 F 3 "~" H 4600 3075 50  0001 C CNN
 	1    4600 3075
@@
 F 0 "JP3" H 3675 5714 50  0000 C CNN
 F 1 "RefToDRL" H 3675 5623 50  0000 C CNN
-F 2 "Connector_PinHeader_1.00mm:PinHeader_1x02_P1.00mm_Vertical" H 3675 5450 50  0001 C CNN
+F 2 "Connector_PinHeader_2.54mm:PinHeader_1x02_P2.54mm_Vertical" H 3675 5450 50  0001 C CNN
 F 3 "~" H 3675 5450 50  0001 C CNN
 	1    3675 5450
@@
 	0    1    1    0
 $EndComp
+Wire Notes Line
+	4000 1750 5700 1750
+Wire Notes Line
+	5700 1750 5700 2375
+Wire Notes Line
+	5700 2375 4000 2375
+Wire Notes Line
+	4000 2375 4000 1750
+$Comp
+L Device:LED D1
+U 1 1 5D238FF7
+P 4300 2050
+F 0 "D1" H 4275 1850 50  0000 C CNN
+F 1 "Green Led" H 4225 1925 50  0000 C CNN
+F 2 "LED_THT:LED_D5.0mm" H 4300 2050 50  0001 C CNN
+F 3 "~" H 4300 2050 50  0001 C CNN
+	1    4300 2050
+	-1   0    0    1
+$EndComp
+$Comp
+L Device:LED D2
+U 1 1 5D239E6B
+P 4975 2050
+F 0 "D2" H 5000 2250 50  0000 C CNN
+F 1 "Blue Led" H 5025 2175 50  0000 C CNN
+F 2 "LED_THT:LED_D5.0mm" H 4975 2050 50  0001 C CNN
+F 3 "~" H 4975 2050 50  0001 C CNN
+	1    4975 2050
+	1    0    0    -1
+$EndComp
+$Comp
+L power:+12V #PWR0124
+U 1 1 5D23ADFA
+P 4100 1975
+F 0 "#PWR0124" H 4100 1825 50  0001 C CNN
+F 1 "+12V" H 4115 2148 50  0000 C CNN
+F 2 "" H 4100 1975 50  0001 C CNN
+F 3 "" H 4100 1975 50  0001 C CNN
+	1    4100 1975
+	1    0    0    -1
+$EndComp
+$Comp
+L power:-12V #PWR0125
+U 1 1 5D23BE77
+P 4775 1975
+F 0 "#PWR0125" H 4775 2075 50  0001 C CNN
+F 1 "-12V" H 4790 2148 50  0000 C CNN
+F 2 "" H 4775 1975 50  0001 C CNN
+F 3 "" H 4775 1975 50  0001 C CNN
+	1    4775 1975
+	1    0    0    -1
+$EndComp
+$Comp
+L power:GND #PWR0126
+U 1 1 5D3403C3
+P 4550 2150
+F 0 "#PWR0126" H 4550 1900 50  0001 C CNN
+F 1 "GND" H 4555 1977 50  0000 C CNN
+F 2 "" H 4550 2150 50  0001 C CNN
+F 3 "" H 4550 2150 50  0001 C CNN
+	1    4550 2150
+	1    0    0    -1
+$EndComp
+$Comp
+L power:GND #PWR0127
+U 1 1 5D3407E1
+P 5225 2150
+F 0 "#PWR0127" H 5225 1900 50  0001 C CNN
+F 1 "GND" H 5230 1977 50  0000 C CNN
+F 2 "" H 5225 2150 50  0001 C CNN
+F 3 "" H 5225 2150 50  0001 C CNN
+	1    5225 2150
+	1    0    0    -1
+$EndComp
+Wire Wire Line
+	4150 2050 4100 2050
+Wire Wire Line
+	4100 2050 4100 1975
+Wire Wire Line
+	4450 2050 4550 2050
+Wire Wire Line
+	4550 2050 4550 2150
+Wire Wire Line
+	4825 2050 4775 2050
+Wire Wire Line
+	4775 2050 4775 1975
+Wire Wire Line
+	5125 2050 5225 2050
+Wire Wire Line
+	5225 2050 5225 2150
+Text Notes 5125 1850 0    50   ~ 10
+Indicator Leds
+Text Notes 6975 6450 0    50   ~ 0
+AD620\nManufacturer: Analogic Devices\nPackage: Lead Plastic Dual In-Line
+Text Notes 8500 6450 0    50   ~ 0
+LM741\nManufacturer: Fairchild Semiconductor\nPackage: Lead Plastic Dual In-Line
 $EndSCHEMATC
